File: Accumulator Base/DCDC.sch (KiCad schematic (older format))
At the start: 12 parts, among them J1 Conn_01x04, U11 QHL300, U9 TEC2-1211WI

Commit message: Accumulator Base layout with no traces
Parts:
- C1: footprint Capacitor_SMD:C_1206_3216Metric -> UVR2V010MED:CAPPRD250W50D655H1250
- C2: footprint Capacitor_SMD:C_1206_3216Metric -> EEV-EB2V100SM:CAPAE1700X1700N
- C3: footprint Capacitor_SMD:C_1206_3216Metric -> Capacitor_SMD:C_0805_2012Metric
- F7: footprint Fuse:Fuseholder_Blade_Mini_Keystone_3568 -> Fuse:Fuseholder_Cylinder-5x20mm_Schurter_0031_8201_Horizontal_Open
- J1: value Conn_01x04 -> Accu Cooling; footprint Connector_PinHeader_2.54mm:PinHeader_1x04_P2.54mm_Vertical -> Connector_Molex:Molex_Mini-Fit_Jr_5566-04A_2x02_P4.20mm_Vertical
- U9: value TEC2-1211WI -> NCS1S1212SC; footprint Converter_DCDC:Converter_DCDC_TRACO_TMR-xxxx_THT -> Converter_DCDC:Converter_DCDC_Murata_NCS1SxxxxSC_THT; symbol Converter_DCDC:TEC2-1211WI -> Converter_DCDC:NCS1S1212SC
Connections:
- net at U11.5 (Sense+): now also RV3.1; no longer RV3.3
- net at U11.7 (Sense+): now also RV3.3; no longer RV3.1
Other:
- note added: "This DCDC turns on/off the QHL300. \n12V in pin 3 will turn the DCDC OFF and if pin 3 is left open it will be ON.\nQHL ON/OFF requires signal referenced off HV-.\nThe control signal will be analogically activated by a switch in the Dash."
- note removed: "This DCDC turns on/off the QHL300. QHL ON/OFF \nrequires signal referenced off HV-."
Changed lines of the file:
@@
 F 0 "F3" V 2053 2700 50  0000 C CNN
 F 1 "5A" V 2144 2700 50  0000 C CNN
-F 2 "Fuse:Fuseholder_Blade_Mini_Keystone_3568" V 2180 2700 50  0001 C CNN
+F 2 "Fuse:Fuseholder_Cylinder-5x20mm_Schurter_0031_8201_Horizontal_Open" V 2180 2700 50  0001 C CNN
 F 3 "~" H 2250 2700 50  0001 C CNN
 	1    2250 2700
@@
 F 0 "C2" H 3878 2496 50  0000 L CNN
 F 1 "10u" H 3878 2405 50  0000 L CNN
-F 2 "Capacitor_SMD:C_1206_3216Metric" H 3700 2450 50  0001 C CNN
+F 2 "EEV-EB2V100SM:CAPAE1700X1700N" H 3700 2450 50  0001 C CNN
 F 3 "~" H 3700 2450 50  0001 C CNN
 	1    3700 2450
@@
 F 0 "C1" H 2828 2496 50  0000 L CNN
 F 1 "1u" H 2828 2405 50  0000 L CNN
-F 2 "Capacitor_SMD:C_1206_3216Metric" H 2650 2450 50  0001 C CNN
+F 2 "UVR2V010MED:CAPPRD250W50D655H1250" H 2650 2450 50  0001 C CNN
 F 3 "~" H 2650 2450 50  0001 C CNN
 	1    2650 2450
@@
 	3000 2700 2650 2700
 $Comp
-L Converter_DCDC:TEC2-1211WI U9
+L Converter_DCDC:NCS1S1212SC U9
 U 1 1 5EC472A5
 P 2800 3350
@@
 AR Path="/5F131378/5EC472A5" Ref="U6"  Part="1"
 F 0 "U6" H 2800 3817 50  0000 C CNN
-F 1 "TEC2-1211WI" H 2800 3726 50  0000 C CNN
-F 2 "Converter_DCDC:Converter_DCDC_TRACO_TMR-xxxx_THT" H 2800 3000 50  0001 C CNN
+F 1 "NCS1S1212SC" H 2800 3726 50  0000 C CNN
+F 2 "Converter_DCDC:Converter_DCDC_Murata_NCS1SxxxxSC_THT" H 2800 3000 50  0001 C CNN
 F 3 "https://www.tracopower.com/products/tec2wi.pdf" H 2800 2850 50  0001 C CNN
 	1    2800 3350
@@
 F 0 "C3" H 4178 3396 50  0000 L CNN
 F 1 "10u" H 4178 3305 50  0000 L CNN
-F 2 "Capacitor_SMD:C_1206_3216Metric" H 4000 3350 50  0001 C CNN
+F 2 "Capacitor_SMD:C_0805_2012Metric" H 4000 3350 50  0001 C CNN
 F 3 "~" H 4000 3350 50  0001 C CNN
 	1    4000 3350
@@
 F 3 "~" H 6250 2450 50  0001 C CNN
 	1    6250 2450
-	-1   0    0    1
+	-1   0    0    -1
 $EndComp
 Wire Wire Line
@@
 AR Path="/5F131378/5EA1EAAD" Ref="J6"  Part="1"
 F 0 "J6" H 9280 2892 50  0000 L CNN
-F 1 "Conn_01x04" H 9280 2801 50  0000 L CNN
-F 2 "Connector_PinHeader_2.54mm:PinHeader_1x04_P2.54mm_Vertical" H 9200 2900 50  0001 C CNN
+F 1 "Accu Cooling" H 9280 2801 50  0000 L CNN
+F 2 "Connector_Molex:Molex_Mini-Fit_Jr_5566-04A_2x02_P4.20mm_Vertical" H 9200 2900 50  0001 C CNN
 F 3 "~" H 9200 2900 50  0001 C CNN
 	1    9200 2900
@@
 Wire Wire Line
 	4000 3100 4750 3100
-Text Notes 2450 3900 0    50   ~ 0
-This DCDC turns on/off the QHL300. QHL ON/OFF \nrequires signal referenced off HV-.
+Text Notes 1700 4500 0    79   ~ 0
+This DCDC turns on/off the QHL300. \n12V in pin 3 will turn the DCDC OFF and if pin 3 is left open it will be ON.\nQHL ON/OFF requires signal referenced off HV-.\nThe control signal will be analogically activated by a switch in the Dash.
 Text Notes 3150 3000 0    50   ~ 0
 transient voltage \nsuppressor diode
