File: Accumulator Base/MCU+Drivers.sch (KiCad schematic (older format))
At the start: 47 parts, among them J20 LCD, Q10 Q_NMOS_GDS, Q11 Q_NMOS_GDS, Q12 Q_NMOS_GDS, Q13 Q_NMOS_GDS, Q14 Q_NMOS_GDS, Q15 Q_NMOS_GDS, Q16 Q_NMOS_GDS, Q17 Q_NMOS_GDS, Q18 Q_NMOS_GDS, Q19 Q_NMOS_GDS, Q20 Q_NMOS_GDS, Q21 Q_NMOS_GDS, Q5 Q_NMOS_GDS, U4 LAUNCHXL-F28379D, U9 LM3670MF

Commit message: Base PCB finished with traces
Connections:
- net +5V: no longer U4.3, U4.35
- net 3.3V: no longer U4.13, U4.45
Changed lines of the file:
@@
 Text GLabel 6550 2600 1    50   Input ~ 0
 3.3V
-Text HLabel 4200 2900 3    50   Input ~ 0
-+5V
 Text HLabel 4100 2900 3    50   Input ~ 0
 GND
@@
 Text HLabel 6950 4750 3    50   Input ~ 0
 +5V
-Text GLabel 6350 2600 1    50   Input ~ 0
-3.3V
 Text GLabel 8800 900  1    50   Input ~ 0
 3.3V
@@
 Text Notes 4750 650  0    50   ~ 0
 Coil model: TFM322512ALMA100MTAA
-Text GLabel 4200 2600 1    50   Input ~ 0
-3.3V
-Text HLabel 6350 2900 3    50   Input ~ 0
-+5V
 Text HLabel 6350 4750 3    50   Input ~ 0
 GND
