File: Battery Monitoring Board/08-14-2020 BMB/Slave Board.kicad_pcb (KiCad board)
At the start: 2 copper layers, 438 x 77.5 mm, 150 parts, among them IC1 LTC6820IMS#PBF, IC2 LTC6804-2, J1 Conn_01x02, J10 Conn_01x02, J11 Conn_01x02, J12 Conn_01x02, J13 Conn_01x08, J14 Conn_01x01, J15 Conn_01x01, J16 Conn_01x01, J17 Conn_01x01, J18 Conn_01x01, J19 Conn_01x01, J2 Conn_01x02, J20 Conn_01x01, J21 Conn_01x01, J22 Conn_01x01, J23 Conn_01x01, J24 Conn_01x01, J25 Conn_01x01, J26 Conn_01x01, J27 Conn_01x04, J3 Conn_01x02, J4 Conn_01x02, J5 Conn_01x02, J6 Conn_01x02, J7 Conn_01x02, J8 Conn_01x02, J9 Conn_01x02, Q1 Q_NPN_BCE, Q10 Q_PMOS_GSD, Q11 Q_PMOS_GSD, Q12 Q_PMOS_GSD, Q13 Q_PMOS_GSD, Q2 Q_PMOS_GSD, Q3 Q_PMOS_GSD, Q4 Q_PMOS_GSD, Q5 Q_PMOS_GSD, Q6 Q_PMOS_GSD, Q7 Q_PMOS_GSD, Q8 Q_PMOS_GSD, Q9 Q_PMOS_GSD, T1 PE-68386NL, U1 MCP2551_CANmodule, U2 MCP2551-I-SN, U3 OKI-78SR-3.3_1.5-W36-C, U4 ISO1050DUB, U5 TMR_1-1212, U6 ARDUINO_MICRO_SHIELD

Commit message: BMB shortened
Parts:
- moved D1 52.2 mm to (121.7, 216.3)
- moved C7 52.1 mm to (121.1, 214.2)
- moved C8 52.1 mm to (117.8, 208.3)
- moved U3 52.1 mm to (123.5, 209.5)
- moved G*** 35.6 mm to (173.7, 214.5)
- moved F13 34.5 mm to (154.6, 249.2), turned to 90 degrees
- moved J26 34.4 mm to (150.0, 250.8)
- moved R19 34.3 mm to (117.4, 198.7)
- moved U2 34.3 mm to (121.2, 200.2)
- moved C12 34.2 mm to (138.5, 218.1)
- moved U5 34.2 mm to (139.8, 222.5)
- moved C10 34.0 mm to (128.6, 190.4)
- moved C13 34.0 mm to (137.7, 190.6)
- moved U4 34.0 mm to (132.2, 196.6)
- moved C11 32.6 mm to (121.3, 218.6)
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Routing:
- net VCC_ISO: track 189.9 -> 159.1 mm
- net VCC: track 63.7 -> 34.9 mm
- net SO: track 183.3 -> 157.3 mm
- net SCK: track 186.3 -> 160.3 mm
- net SI: track 181.5 -> 155.6 mm
- net CS: track 193.1 -> 167.3 mm
- net +5V: track 148.3 -> 122.7 mm, vias 10 -> 8
- net Cell12: track 304.7 -> 280.7 mm
- net T11: track 194.0 -> 172.5 mm, vias 5 -> 4
- net T0: track 259.1 -> 238.2 mm
- net PWM_Fans: track 25.6 -> 6.32 mm, vias 2 -> 0
- net Sens_Fans: track 23.6 -> 6.13 mm, vias 3 -> 0
- net DCDC+: track 19.8 -> 6.08 mm, vias 2 -> 0
- net C0: track 329.8 -> 316.1 mm, vias 10 -> 12
- net C1: track 320.5 -> 308.7 mm, vias 6 -> 8
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Other:
- board size 438 x 77.5 mm -> 412.7 x 77.5 mm
